File: robotArm/robotArm.kicad_pcb (KiCad board)
At the start: 4 copper layers, 127 x 66 mm, 30 parts, among them J1 Barrel_Jack, J2 Conn_01x16_Pin, J3 Conn_01x04, J4 Conn_01x04, J5 Conn_01x04, J6 Conn_01x04, U2 TMC2209_SILENTSTEPSTICK, U4 TMC2209_SILENTSTEPSTICK, U5 TMC2209_SILENTSTEPSTICK, U6 74HC165

Commit message: Moved GND plane from B.cu to in2.cu
Parts:
- D5: value IX1 -> D5
Routing:
- net GND: track 253.8 -> 37.4 mm
- net +12V: track 166.1 -> 182.6 mm, vias 0 -> 1
- net UART2_TX: track 140.7 -> 131.4 mm, vias 0 -> 3
- net /M2-1A: track 17.7 -> 8.50 mm
- net /M4-1A: track 8.54 -> 17.7 mm
- net /M3-1B: track 11.9 -> 21.0 mm, vias 1 -> 0
- net /M1-2B: track 19.3 -> 10.6 mm
- net /M3-2B: track 11.8 -> 18.8 mm
- net +3.3V: track 320.2 -> 313.4 mm, vias 1 -> 0
- net DIR_2: track 57.4 -> 64.2 mm, vias 2 -> 1
- net /M2-2B: track 24.9 -> 18.9 mm
- net D3: track 23.0 -> 28.8 mm
- net Net-(J4-2B): track 17.4 -> 11.8 mm
- net Net-(D6-K): track 48.6 -> 43.1 mm, vias 1 -> 0
- net D0: track 53.0 -> 48.0 mm
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- added copper zone on In2.Cu, net GND
- removed copper zone on B.Cu, net GND
Other:
- board text added: "12VDC"
- board text added: "4DoF Robot Control (C) Turnimator Cyberdelix 2026 Jan Atle Ramsli"
- board text added: "DIAG1"
- board text added: "DIAG2"
- board text added: "DIAG3"
- board text added: "DIAG4"
- board text removed: "Turnimator Cyberdelix (C) Jan Atle Ramsli 2026"
