File: robotArm/endstop_section.kicad_sch (KiCad schematic)
At the start: 15 parts, among them J2 ENDSTOP INPUTS, U3 74HC245, U6 74HC165, U9 74LS279

Commit message: Attempt 2.1
Parts:
- removed J2: ENDSTOP INPUTS, Connector_PinHeader_2.54mm:PinHeader_1x16_P2.54mm_Vertical, symbol Connector:Conn_01x16_Pin
- removed R1: R, Resistor_THT:R_Axial_DIN0204_L3.6mm_D1.6mm_P2.54mm_Vertical, symbol Device:R
- added C1, C2, C3, C5: 47μ, Capacitor_THT:CP_Radial_D5.0mm_P2.50mm, symbol Device:C
- added D2: USR2, LED_THT:LED_D5.0mm, symbol Device:LED
- added D3: USR1, LED_THT:LED_D5.0mm, symbol Device:LED
- added D4: USR0, LED_THT:LED_D5.0mm, symbol Device:LED
- added D5: ES3, LED_THT:LED_D5.0mm, symbol Device:LED
- added D6: ES2, LED_THT:LED_D5.0mm, symbol Device:LED
- added D7: ES1, LED_THT:LED_D5.0mm, symbol Device:LED
- added D8: ES0, LED_THT:LED_D5.0mm, symbol Device:LED
- added R11, R12, R13, R14, R15, R16, R17: 330Ω, Resistor_THT:R_Axial_DIN0204_L3.6mm_D1.6mm_P2.54mm_Vertical, symbol Device:R
- D1: value LED -> USR3; footprint (none) -> LED_THT:LED_D5.0mm
- U3: footprint (none) -> Package_DIP:DIP-20_W7.62mm
- U9: footprint (none) -> Package_DIP:DIP-16_W7.62mm
Connections:
- net +3.3V: now also U3.1 (A->B), U9.16 (VCC), C1.1, C2.1, C3.1, C5.1
- net EN_DRV1: now also R17.1; no longer R10.1
- net EN_DRV2: now also R16.1
- net EN_DRV3: now also R15.1
- net EN_DRV4: now also R14.1
- net GND: now also U3.19 (CE), U6.10 (DS), U6.15 (~{CE}), U6.8 (GND), U9.8 (GND), C1.2, C2.2, C3.2, C5.2; no longer D1.1 (K)
- net USR0: now also U3.6 (A4)
- net USR1: now also U3.7 (A5)
- net USR2: now also U3.8 (A6)
- net USR3: now also U3.9 (A7)
- net RESET_DRV: now reaches U9.1 (~{R})
- net RESET_DRV: now also U9.10 (~{R}), U9.14 (~{R}), U9.5 (~{R})
- net at U3.11 (B7): now also R10.1
- net at U3.12 (B6): now also R11.1
- net at U3.13 (B5): now also R12.1
- net at U3.14 (B4): now also R13.1
- new net: D1.1 (K), D2.1 (K), D3.1 (K), D4.1 (K), D5.1 (K), D6.1 (K), D7.1 (K), D8.1 (K)
- new net: D2.2 (A), R11.2
- new net: D8.2 (A), R17.2
- new net: D5.2 (A), R14.2
- new net: D7.2 (A), R16.2
- new net: D4.2 (A), R13.2
- new net: D6.2 (A), R15.2
- new net: D3.2 (A), R12.2
- no-connect marks 1 -> 5
Other:
- note added: "Decoupling IC"
- note added: "End stops and user buttons pull these to ground"
- note added: "Output low=normal operation"
- note removed: "Endstop switches ES0->D0, ES1->D1 ... USR3->D7"
- moved on the sheet: D1, R10, U9A, U9B, U9C, U9D, U9E

Commit message: Added END-EFFECTOR
Not yet sent to JLCPCB
Connections:
- no-connect marks 5 -> 3
Changed lines of the file:
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@@
-	)
-	(no_connect
-		(at 173.99 35.56)
 	)
 	(no_connect
@@
 		(at 52.07 147.32)
 	)
-	(no_connect
-		(at 232.41 35.56)
-	)
 	(wire
